File: docs/engineering/rvb22/candidate/cad/GR86_CCA_RevB.kicad_pcb (KiCad board)
At the start: 4 copper layers, 88.3 x 61.3 mm, 199 parts, among them J201 TC2030-IDC-NL / UART, J202 RESET — short to reset, J203 BOOT — hold low on reset, J401 U.FL-R-SMT-1(80), Q101 STD25NF20 /200V, U101 LTC4367HMS8#WTRPBF, U121 LM5164DDAR, U151 LM63615DQPWPRQ1, U201 ESP32-S3-WROOM-1-N8R2, U202 TPS3808G33-Q1 3.07V RESET, U301 TCAN3403DRBRQ1, U401 PA1616D, U402 SN74LVC2G125DCUR, U403 MIC5504-3.3YM5-TR, U404 SN74LVC2G125DCUR, U501 TPS26600PWPR, U502 OPA2333AIDR

Commit message: I28: automotive-qualify 5V buck and document power signoff
Parts:
- U121: value LM5164DDAR -> LM5164QDDARQ1

Commit message: Complete I32 recovery and 160 MHz firmware closure
Parts:
- added C159: 33n /100V C0G 5% CT, RevB:I32_FINISHED_C159, B.Cu at (44.3, 0.70)
- added C161: 100n /50V X7R ISO INPUT, RevB:I32_FINISHED_C161, B.Cu at (40.6, 4.50)
- added C162: 470u /10V POLYMER INPUT, RevB:I32_FINISHED_C162, F.Cu at (49.0, -5.00)
- added C165: 220n /50V X7R EN DELAY, RevB:I32_FINISHED_C165, F.Cu at (27.0, -0.50)
- added C166: 68n /100V C0G 5% BULK CT, RevB:I32_FINISHED_C166, B.Cu at (85.8, -3.00)
- added C167: 1u /16V X7R BULK INPUT, RevB:I32_FINISHED_C167, B.Cu at (78.5, -0.40)
- added D105: SMCJ110A /RAW OV CLAMP, RevB:D_SMC, F.Cu at (27.0, 44.0)
- added Q152: DMG2302UKQ /DISCHARGE, RevB:I32_FINISHED_Q152, F.Cu at (46.0, 44.0)
- added Q153: DMG2302UKQ /DISCHARGE, RevB:I32_FINISHED_Q153, F.Cu at (50.0, 44.0)
- added R159: 47k /1% PG PULLUP, RevB:I32_FINISHED_R159, F.Cu at (46.0, -1.50)
- added R160: 6.34k /0.02% SNS TOP, RevB:I32_FINISHED_R160, F.Cu at (27.0, -7.50)
- added R161: 1k /0.02% SNS BOTTOM, RevB:I32_FINISHED_R161, F.Cu at (30.5, -7.50)
- added R162: 4.7k /0.02% ISO EN TOP, RevB:I32_FINISHED_R162, F.Cu at (27.0, -4.00)
- added R163: 1k /0.02% ISO EN BOTTOM, RevB:I32_FINISHED_R163, F.Cu at (30.5, -4.00)
- added R164: 4.7k /DISCHARGE GATE FEED, RevB:I32_FINISHED_R164, F.Cu at (48.0, 48.2)
- added R165: 4.7R /1.5W PULSE DISCHARGE, RevB:I32_FINISHED_R165, F.Cu at (39.5, 44.0)
- added R166: 330k /1% U151 EN DIVIDER, RevB:I32_FINISHED_R166, F.Cu at (35.0, -7.50)
- added R167: 330k /1% U151 EN DIVIDER, RevB:I32_FINISHED_R167, F.Cu at (39.0, -7.50)
- added R168: 1k /1% RESERVOIR BLEED, RevB:I32_FINISHED_R168, B.Cu at (86.3, 2.00)
- added R169: 3.01k /0.02% BULK EN TOP, RevB:I32_FINISHED_R169, B.Cu at (80.0, 2.00)
- added R170: 1k /0.02% BULK EN BOTTOM, RevB:I32_FINISHED_R170, B.Cu at (83.3, 2.00)
- added R204: 100k /1% RESET DELAY, RevB:I32_FINISHED_R204, B.Cu at (75.6, 6.90)
- added TP154: TP_ISO_ENABLE, RevB:I32_FINISHED_TP154, F.Cu at (33.0, -1.00)
- added U152: TPS22953-Q1 REVERSE BLOCKING, RevB:I32_FINISHED_U152, B.Cu at (43.6, 4.80)
- added U153: TPS22953-Q1 BULK CHARGER, RevB:I32_FINISHED_U153, B.Cu at (79.1, -3.50)
- C206: value 470u /6.3V POLYMER -> 680u /6.3V POLYMER
- D101: value S5D /200V 5A -> S5J /600V REVERSE BLOCK
- R101: value 6.81k /1W -> 12.1k /1W CTRL SURGE FEED
- R151: footprint RevB:R_1206_3216Metric -> RevB:I32_FINISHED_R151
- R155: footprint RevB:R_0603_1608Metric_RVB22_R155 -> RevB:I32_FINISHED_R155
- R156: value 4.99k /0.02% 2ppm FB BOTTOM -> 5.05k /0.02% 2ppm FB BOTTOM; footprint RevB:R_0603_1608Metric_RVB22_R156 -> RevB:I32_FINISHED_R156
- R158: value 82m /1% BULK DAMPING -> 300m /1% BULK DAMPING; footprint RevB:WSLP0603_MANUFACTURER -> RevB:I32_FINISHED_R158
- moved R158 23.6 mm to (82.7, -4.00), turned to 90 degrees
- moved R156 16.8 mm to (41.2, 10.8)
- moved R155 16.1 mm to (44.5, 10.8)
- moved R151 10.3 mm to (38.6, 1.70)
Connections:
- R151 pad 2: 3V3_VIN -> 3V3_ISO_IN
- R158 pad 1: +3V3 -> 3V3_BULK_SWITCHED
- U151 pad 11: 3V3_VIN -> 3V3_BUCK_ENABLE
- U202 pad 4: unconnected-(U202-CT-Pad4) -> SUP_RESET_DELAY
Routing:
- net 3V3_ENABLE: track 0.00 -> 165.2 mm, vias 0 -> 3
- net 3V3_VIN: track 11.7 -> 140.3 mm, vias 0 -> 4
- net 3V3_FB_ADJ: track 64.0 -> 7.00 mm, vias 4 -> 0
- net +3V3: track 338.9 -> 393.8 mm, vias 11 -> 15
- net 3V3_SOURCE: track 72.9 -> 116.9 mm, vias 4 -> 6
- net GND: track 179.6 -> 221.4 mm, vias 156 -> 171
- net 3V3_BUCK_ENABLE: track 0.00 -> 41.5 mm, vias 0 -> 2
- net 3V3_ISO_ENABLE: track 0.00 -> 35.8 mm, vias 0 -> 2
- net +5V: track 115.4 -> 147.0 mm, vias 8 -> 9
- net 3V3_ISO_SNS: track 0.00 -> 28.3 mm, vias 0 -> 2
- net REV_BLOCKED_12V: track 25.7 -> 53.2 mm, vias 2 -> 3
- net 3V3_BULK_DAMPED: track 32.0 -> 15.7 mm
- net 3V3_BULK_ENABLE: track 0.00 -> 14.8 mm, vias 0 -> 2
- net SUP_RESET_DELAY: track 0.00 -> 13.6 mm, vias 0 -> 2
- net 3V3_DISCHARGE_GATE: track 0.00 -> 11.3 mm
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Other:
- board text added: "+"
